Commit message: Changed TF publisher from static_transform_publisher to robot_state_publisher

File: description/robot.urdf (robot description, URDF)
Before this commit: robot robot, 7 links, 6 joints
Links:
- added link imu_link; visual box size=0.035 0.035 0.010
Joints:
- added joint imu_link_joint: type fixed, parent base_link, child imu_link, origin xyz=0.3 0.0 0.095, axis 0 0 1
- joint base_footprint_joint: origin xyz=0 0 -0.3465 -> xyz=0 0 0
- joint caster_joint: origin xyz=-0.32 0.0 -0.305 -> xyz=-0.32 0.0 0.0505
- joint gps_joint: origin xyz=-0.32 0.0 0.30 -> xyz=-0.32 0.0 0.65
- joint laser_joint: origin xyz=0.32 0.0 0.275 -> xyz=0.32 0.0 0.625
- joint left_wheel_joint: origin xyz=0.3 0.24 -0.25 rpy=0 0 0 -> xyz=0.3 0.24 0.095 rpy=0 0 0
- joint right_wheel_joint: origin xyz=0.3 -0.24 -0.25 -> xyz=0.3 -0.24 0.095

Commit message: Fixed TF relationship

File: description/robot.urdf (robot description, URDF)
Before this commit: robot robot, 8 links, 7 joints
Joints:
- joint base_footprint_joint: child base_footprint -> base_link; origin xyz=0 0 0 -> xyz=0 0 0.35; parent base_link -> base_footprint
- joint caster_joint: origin xyz=-0.32 0.0 0.0505 -> xyz=-0.32 0.0 -0.305
- joint gps_joint: origin xyz=-0.32 0.0 0.65 -> xyz=-0.32 0.0 0.30
- joint imu_link_joint: origin xyz=0.3 0.0 0.095 -> xyz=0.3 0.0 0.0
- joint laser_joint: origin xyz=0.32 0.0 0.625 -> xyz=0.32 0.0 0.275
- joint left_wheel_joint: origin xyz=0.3 0.24 0.095 rpy=0 0 0 -> xyz=0.3 0.24 -0.25 rpy=0 0 0
- joint right_wheel_joint: origin xyz=0.3 -0.24 0.095 -> xyz=0.3 -0.24 -0.25

Commit message: Fixed TF relationship

File: description/robot.urdf (robot description, URDF)
Before this commit: robot robot, 8 links, 7 joints
Joints:
- joint imu_link_joint: origin xyz=0.3 0.0 0.0 -> xyz=0.3 0.0 -0.25
- joint laser_joint: origin xyz=0.32 0.0 0.275 -> xyz=0.32 0.0 0.275 rpy=3.14 0 3.14

Commit message: Fixed robot wheelbase in robot URDF

File: description/robot.urdf (robot description, URDF)
Before this commit: robot robot, 8 links, 7 joints
Joints:
- joint left_wheel_joint: origin xyz=0.3 0.24 -0.25 rpy=0 0 0 -> xyz=0.3 0.2435 -0.25 rpy=0 0 0
- joint right_wheel_joint: origin xyz=0.3 -0.24 -0.25 -> xyz=0.3 -0.2435 -0.25

Commit message: Updated robot URDF

File: description/robot.urdf (robot description, URDF)
Before this commit: robot robot, 8 links, 7 joints
Links:
- link base_link: geometry collision box size=0.74 0.42 0.51; visual box size=0.74 0.42 0.51
Joints:
- joint gps_joint: origin xyz=-0.32 0.0 0.30 -> xyz=-0.255 0.0 0.30
- joint laser_joint: origin xyz=0.32 0.0 0.275 rpy=3.14 0 3.14 -> xyz=0.265 0.0 0.275 rpy=3.14 0 3.14

Commit message: Updated robot URDF

File: description/robot.urdf (robot description, URDF)
Before this commit: robot robot, 8 links, 7 joints
Joints:
- joint imu_link_joint: origin xyz=0.3 0.0 -0.25 -> xyz=0.275 0.0 -0.25
- joint left_wheel_joint: origin xyz=0.3 0.2435 -0.25 rpy=0 0 0 -> xyz=0.275 0.2435 -0.25
- joint right_wheel_joint: origin xyz=0.3 -0.2435 -0.25 -> xyz=0.275 -0.2435 -0.25
