Commit message: Minor fix

File: description/robot_camera.urdf (robot description, URDF)
Before this commit: robot robot, 9 links, 8 joints
Joints:
- joint camera_joint: origin xyz=0.375 0.0 -0.012 -> xyz=0.375 0.0 0.010

Commit message: minor fix

File: description/robot_camera.urdf (robot description, URDF)
Before this commit: robot robot, 9 links, 8 joints
Joints:
- joint camera_joint: origin xyz=0.375 0.0 0.010 -> xyz=0.375 0.0 0.090
